File: circuits/28byj_controller/28byj_controller.kicad_pcb (KiCad board)
At the start: 2 copper layers, 50 x 50 mm, 17 parts, among them J1 INPUT, J2 5V, M1 28BYJ-48_Stepper, M2 28BYJ-48_Stepper, U1 74HC595, U2 ULN2803A

Commit message: Big changes
Other:
- net class Default removed
