File: circuits/x27_controller/x27_controller.kicad_pcb (KiCad board)
At the start: 2 copper layers, 50 x 50 mm, 19 parts, among them J1 INPUT, J2 5V, M1 x27_Stepper, U1 74HC595

Commit message: Big changes
Routing:
- net Net-(M1-Pad4): track 12.2 -> 21.5 mm
- net Net-(M1-Pad3): track 9.52 -> 17.8 mm
- net Net-(M1-Pad2): track 17.3 -> 10.0 mm
- net Net-(M1-Pad1): track 12.8 -> 18.6 mm
- net Net-(R10-Pad1): track 22.4 -> 25.9 mm
- net +5V: track 60.2 -> 57.2 mm, vias 2 -> 1
Other:
- net class Default removed
