File: circuits/base_controller/ESP32.kicad_sch (KiCad schematic)
At the start: 9 parts

Commit message: Big updates
Parts:
- removed R12, R13, R14, R15: 10 K, Resistor_SMD:R_0805_2012Metric_Pad1.20x1.40mm_HandSolder, symbol Device:R
- added J1: JTAG, Connector_PinHeader_2.54mm:PinHeader_2x05_P2.54mm_Vertical, symbol Connector:Conn_ARM_JTAG_SWD_10
- C1: renamed from C?; value (none) -> 10 uF; footprint (none) -> Capacitor_SMD:C_0805_2012Metric_Pad1.18x1.45mm_HandSolder
- C2: renamed from C?; value (none) -> 0.1 uF; footprint (none) -> Capacitor_SMD:C_0805_2012Metric_Pad1.18x1.45mm_HandSolder
- U1: renamed from U?; value (none) -> ESP32-WROOM-32; footprint (none) -> RF_Module:ESP32-WROOM-32
- renumbered R10 to R1, R11 to R2
Connections:
- net EN is gone; now on net +3V3: U1.3 (EN)
- net +3V3: now also J1.1 (VTref)
- net Earth: now also J1.10 (~{RESET}), J1.3 (GND), J1.5 (GND), J1.9 (GNDDetect)
- net MTCK: now also J1.4 (SWDCLK/TCK)
- net MTDI: now also J1.8 (NC/TDI)
- net MTDO: now also J1.6 (SWO/TDO)
- net MTMS: now also J1.2 (SWDIO/TMS)
- net DEVID_0: no longer names the net of U1.4 (SENSOR_VP)
- net DEVID_1: no longer names the net of U1.5 (SENSOR_VN)
- net DEVID_2: no longer names the net of U1.6 (IO34)
- net DEVID_3: no longer names the net of U1.7 (IO35)
- net RXD0: no longer names the net of U1.34 (RXD0/IO3)
- net TXD0: no longer names the net of U1.35 (TXD0/IO1)
- no-connect marks 6 -> 12
