File: circuits/base_controller/Headers.kicad_sch (KiCad schematic)
At the start: 14 parts, among them J1 OUTPUT, J2 INPUT, J3 3V3, J4 5V

Commit message: Big updates
Parts:
- removed JP1, JP6: 0, Connector_PinHeader_2.54mm:PinHeader_1x03_P2.54mm_Vertical, symbol base_controller-rescue:Jumper_3_Open-Jumper
- removed JP2, JP7: 1, Connector_PinHeader_2.54mm:PinHeader_1x03_P2.54mm_Vertical, symbol base_controller-rescue:Jumper_3_Open-Jumper
- removed JP3, JP8: 2, Connector_PinHeader_2.54mm:PinHeader_1x03_P2.54mm_Vertical, symbol base_controller-rescue:Jumper_3_Open-Jumper
- removed JP4, JP9: 3, Connector_PinHeader_2.54mm:PinHeader_1x03_P2.54mm_Vertical, symbol base_controller-rescue:Jumper_3_Open-Jumper
- removed JP5: 4, Connector_PinHeader_2.54mm:PinHeader_1x03_P2.54mm_Vertical, symbol base_controller-rescue:Jumper_3_Open-Jumper
- added D1, D2, D3, D4, D5: DIODE, Diode_SMD:D_0805_2012Metric_Pad1.15x1.40mm_HandSolder, symbol pspice:DIODE
- added R4, R5, R6, R7, R8: 4.7 k, Resistor_SMD:R_0805_2012Metric_Pad1.20x1.40mm_HandSolder, symbol Device:R
- added SW1: DEV_CLASS, Button_Switch_THT:SW_DIP_SPSTx05_Slide_9.78x14.88mm_W7.62mm_P2.54mm, symbol Switch:SW_DIP_x05
- renumbered J1 to J2, J2 to J3, J3 to J4, J4 to J5, R9 to R3
Connections:
- net +3V3: now also R4.1, R5.1, R6.2, R7.1, R8.2
- net DEVCL_0: now also R7.2, SW1.10
- net DEVCL_1: now also R5.2, SW1.9
- net DEVCL_2: now also R4.2, SW1.8
- net DEVCL_3: now also R8.1, SW1.7
- net DEVCL_4: now also R6.1, SW1.6
- net Earth: now also D1.2 (A), D2.2 (A), D3.2 (A), D4.2 (A), D5.2 (A)
- new net: D3.1 (K), SW1.3
- new net: D5.1 (K), SW1.5
- new net: D4.1 (K), SW1.4
- new net: D2.1 (K), SW1.2
- new net: D1.1 (K), SW1.1
