File: circuits/base_controller/USB_Programmer.kicad_sch (KiCad schematic)
At the start: 12 parts, among them J5 USB_B_Micro, Q1 S8050, U2 CP2102N-A01-GQFN24

Commit message: Big updates
Parts:
- removed C5: 4.7 uF, Capacitor_SMD:C_0805_2012Metric_Pad1.18x1.45mm_HandSolder, symbol pspice:C
- removed C6: 0.1 uF, Capacitor_SMD:C_0805_2012Metric_Pad1.18x1.45mm_HandSolder, symbol pspice:C
- removed D1: SP0503BAHT, Package_TO_SOT_SMD:SOT-143, symbol Power_Protection:SP0503BAHT
- removed J5: USB_B_Micro, Connector_USB:USB_Micro-B_Amphenol_10118194_Horizontal, symbol Connector:USB_B_Micro
- removed Q1: S8050, Package_TO_SOT_SMD:SOT-23, symbol Transistor_BJT:S8050
- removed R3, R6, R7: 1 K, Resistor_SMD:R_0805_2012Metric_Pad1.20x1.40mm_HandSolder, symbol Device:R
- removed R4: 22.1 K, Resistor_SMD:R_0805_2012Metric_Pad1.20x1.40mm_HandSolder, symbol Device:R
- removed R5: 47.5 K, Resistor_SMD:R_0805_2012Metric_Pad1.20x1.40mm_HandSolder, symbol Device:R
- removed R8: 10 K, Resistor_SMD:R_0805_2012Metric_Pad1.20x1.40mm_HandSolder, symbol Device:R
- removed U2: CP2102N-A01-GQFN24, Package_DFN_QFN:QFN-24-1EP_4x4mm_P0.5mm_EP2.6x2.6mm, symbol base_controller-rescue:CP2102N-A01-GQFN24-Interface_USB
Connections:
- no-connect marks 10 -> 0
